Commit message: correcting errors after restructuring

File: urdf/car.urdf (robot description, URDF)
Before this commit: robot robot_name, 7 links, 6 joints
Links:
- link car_body: geometry visual mesh filename=/home/jram/project_car_urdf/assets/car.obj
- link wheel_front_left: geometry visual mesh filename=/home/jram/project_car_urdf/assets/wheel.obj scale=1.0
- link wheel_front_right: geometry visual mesh filename=/home/jram/project_car_urdf/assets/wheel.obj scale=1.0
- link wheel_rear_left: geometry visual mesh filename=/home/jram/project_car_urdf/assets/wheel.obj
- link wheel_rear_right: geometry visual mesh filename=/home/jram/project_car_urdf/assets/wheel.obj

Commit message: changed so that it works in rviz

File: urdf/car.urdf (robot description, URDF)
Before this commit: robot robot_name, 7 links, 6 joints
Links:
- link car_body: geometry visual mesh filename=file:///home/jram/project_car_urdf/assets/car.obj
- link wheel_front_left: geometry visual mesh filename=file:///home/jram/project_car_urdf/assets/wheel.obj
- link wheel_front_right: geometry visual mesh filename=file:///home/jram/project_car_urdf/assets/wheel.obj
- link wheel_rear_left: geometry visual mesh filename=file:///home/jram/project_car_urdf/assets/wheel.obj
- link wheel_rear_right: geometry visual mesh filename=file:///home/jram/project_car_urdf/assets/wheel.obj
Joints:
- joint car_to_front_right_turner: limit (none) -> lower=-0.44 upper=0.44 effort=100 velocity=1.0
- joint joint_car_right_turner_to_wheel_front_right: type revolute -> continuous
- joint joint_car_to_front_wheel_left_turner: limit (none) -> lower=-0.44 upper=0.44 effort=100 velocity=1.0
- joint joint_car_to_left_turner_to_wheel_front_left: type revolute -> continuous
- joint joint_car_to_rear_wheel_left: type revolute -> continuous
- joint joint_car_to_rear_wheel_right: type revolute -> continuous

Commit message: corrected the mistake in urdf file by changing file:// to packge://

File: urdf/car.urdf (robot description, URDF)
Before this commit: robot robot_name, 7 links, 6 joints
Links:
- link car_body: geometry visual mesh filename=package://project_car_urdf/assets/car.obj
- link wheel_front_left: geometry visual mesh filename=package://project_car_urdf/assets/wheel.obj
- link wheel_front_right: geometry visual mesh filename=package://project_car_urdf/assets/wheel.obj
- link wheel_rear_left: geometry visual mesh filename=package://project_car_urdf/assets/wheel.obj
- link wheel_rear_right: geometry visual mesh filename=package://project_car_urdf/assets/wheel.obj

Commit message: changed joint name to be consistent

File: urdf/car.urdf (robot description, URDF)
Before this commit: robot robot_name, 7 links, 6 joints
Joints:
- removed joint car_to_front_right_turner
- added joint joint_car_to_front_right_turner: type revolute, parent car_body, child front_wheel_right_turn, origin xyz=+0.9 1.02 0.2, axis 0 0 1, limit lower=-0.44 upper=0.44 effort=100 velocity=1.0

Commit message: made the car to appear in gazebo and added 1 to the z axis of the car

File: urdf/car.urdf (robot description, URDF)
Before this commit: robot robot_name, 7 links, 6 joints
Links:
- link car_body: mass None -> 50.0; geometry collision mesh filename=package://project_car_urdf/assets/car.obj; visual mesh filename=package://project_car_urdf/assets/car.obj
- link front_wheel_left_turn: mass None -> 5.0; geometry collision box size=0.3 0.3 0.3; visual box size=0.3 0.3 0.3
- link front_wheel_right_turn: mass None -> 5.0; geometry visual box size=0.3 0.3 0.3; visual box size=0.3 0.3 0.3
- link wheel_front_left: mass None -> 5.0; geometry collision mesh filename=package://project_car_urdf/assets/wheel.obj; visual mesh filename=package://project_car_urdf/assets/wheel.obj
- link wheel_front_right: mass None -> 5.0; geometry collision mesh filename=package://project_car_urdf/assets/wheel.obj; visual mesh filename=package://project_car_urdf/assets/wheel.obj
- link wheel_rear_left: mass None -> 5.0; geometry collision mesh filename=package://project_car_urdf/assets/wheel.obj; visual mesh filename=package://project_car_urdf/assets/wheel.obj
- link wheel_rear_right: mass None -> 5.0; geometry collision mesh filename=package://project_car_urdf/assets/wheel.obj; visual mesh filename=package://project_car_urdf/assets/wheel.obj
Joints:
- joint joint_car_to_front_right_turner: origin xyz=+0.9 1.02 0.2 -> xyz=+0.9 1.02 1.2
- joint joint_car_to_front_wheel_left_turner: origin xyz=-0.9 1.02 0.2 -> xyz=-0.9 1.02 1.2
- joint joint_car_to_rear_wheel_left: origin xyz=-0.9 -1.05 0.2 -> xyz=-0.9 -1.05 1.2
- joint joint_car_to_rear_wheel_right: origin xyz=+0.9 -1.05 0.2 -> xyz=+0.9 -1.05 1.2

Commit message: last commit ig

File: urdf/car.urdf (robot description, URDF)
Before this commit: robot robot_name, 7 links, 6 joints
Joints:
- joint joint_car_to_front_right_turner: mimic (none) -> joint=joint_car_to_front_wheel_left_turner
- joint joint_car_to_rear_wheel_right: mimic (none) -> joint=joint_car_to_rear_wheel_left

Commit message: added camera data to rviz

File: urdf/car.urdf (robot description, URDF)
Before this commit: robot robot_name, 7 links, 6 joints
Links:
- added link camera_link, mass 1e-5; collision box size=0.05 0.05 0.05; visual box size=0.05 0.05 0.05
Joints:
- added joint camera_joint: type fixed, parent car_body, child camera_link, origin xyz=0 1.2 2 rpy=0 0 1.5707, axis 0 1 0

Commit message: corrected the car urdf to use simple cylinder for collision mesh and renamed the car in urdf to lamboorgini

File: urdf/car.urdf (robot description, URDF)
Before this commit: robot robot_name, 8 links, 7 joints
Links:
- link front_wheel_right_turn: geometry collision box size=0.3 0.3 0.3; visual box size=0.3 0.3 0.3
- link wheel_front_left: geometry collision cylinder length=0.3 radius=0.46; visual mesh filename=package://project_car_urdf/assets/wheel.obj
- link wheel_front_right: geometry collision cylinder length=0.3 radius=0.46; visual mesh filename=package://project_car_urdf/assets/wheel.obj
- link wheel_rear_left: geometry collision cylinder length=0.3 radius=0.46; visual mesh filename=package://project_car_urdf/assets/wheel.obj
- link wheel_rear_right: geometry collision cylinder length=0.3 radius=0.46; visual mesh filename=package://project_car_urdf/assets/wheel.obj
